Commit message: session 3

File: session3/first_robot_description/urdf/first_robot.urdf (robot description, URDF)
Before this commit: robot first_robot, 5 links, 4 joints
Links:
- link base_link: mass None -> 5; geometry collision box size=0.6 0.4 0.2; visual box size=0.6 0.4 0.2
- link cylinder2_link: mass None -> 1; geometry collision cylinder length=0.05 radius=0.1; visual cylinder length=0.05 radius=0.1
- link cylinder_link: mass None -> 1; geometry collision cylinder length=0.05 radius=0.1; visual cylinder length=0.05 radius=0.1
- link sphere_link: mass None -> 0.5; geometry collision sphere radius=0.05; visual sphere radius=0.05
